Commit message: Changes link/joint names according to FAROS norms

File: urdf/lwr.urdf.xacro (robot description, xacro)
@@ -22,12 +22,12 @@
    <xacro:property name="f5" value="${friction_factor*0.1}"/>
    <xacro:property name="f6" value="${friction_factor*0.1}"/>
-   <xacro:macro name="lwr" params="parent *origin ">
+   <xacro:macro name="lwr" params="parent *origin robot_name:=^|lwr">
       <!-- joint between {parent} and lwr_0_link -->
       <joint name="joint_base" type="fixed">
          <xacro:insert_block name="origin" />
          <parent link="${parent}" />
-         <child link="link_0" />
-      </joint>
-      <link name="link_0">
+         <child link="F_RB${robot_name}" />
+      </joint>
+      <link name="F_RB${robot_name}">
           <inertial>
             <origin
@@ -59,7 +59,7 @@
       </link>
       <!-- joint between lwr_0_link and lwr_1_link -->
-      <joint name="joint_0" type="revolute">
-         <parent link="link_0" />
-         <child link="link_1" />
+      <joint name="${robot_name}_joint_0" type="revolute">
+         <parent link="F_RB${robot_name}" />
+         <child link="F_R${robot_name}_1" />
          <limit lower="${-170 * M_PI / 180}" upper="${170 * M_PI / 180}" effort="${effort_scale * 200}" velocity="${velocity_scale * 112.5 * M_PI / 180}" />
          <dynamics friction="${f0}" damping="${d0}"/>
@@ -67,5 +67,5 @@
          <axis xyz="0 0 1" />
       </joint>
-      <link name="link_1">
+      <link name="F_R${robot_name}_1">
           <inertial>
             <origin
@@ -97,7 +97,7 @@
       </link>
       <!-- joint between lwr_1_link and lwr_2_link -->
-      <joint name="joint_1" type="revolute">
-         <parent link="link_1" />
-         <child link="link_2" />
+      <joint name="${robot_name}_joint_1" type="revolute">
+         <parent link="F_R${robot_name}_1" />
+         <child link="F_R${robot_name}_2" />
          <limit lower="${-120 * M_PI / 180}" upper="${120 * M_PI / 180}" effort="${effort_scale * 200}" velocity="${velocity_scale * 112.5 * M_PI / 180}" />
          <dynamics friction="${f1}" damping="${d1}"/>
@@ -105,19 +105,19 @@
          <axis xyz="0 -1 0" />
       </joint>
-      <link name="link_2">
-    <inertial>
-      <origin
-        xyz="1.26774962153076E-06 -0.032746486541291 0.0736556727355962"
-        rpy="0 0 0" />
-        <mass
-          value="2.30343543179071" />
-      <inertia
-        ixx="0.0142348526057094"
-        ixy="-3.73763310100809E-08"
-        ixz="1.70703603169075E-07"
-        iyy="0.0141319978448755"
-        iyz="0.00228090337255746"
-        izz="0.00424792208583136" />
-    </inertial>
+      <link name="F_R${robot_name}_2">
+         <inertial>
+            <origin
+            xyz="1.26774962153076E-06 -0.032746486541291 0.0736556727355962"
+            rpy="0 0 0" />
+            <mass
+               value="2.30343543179071" />
+            <inertia
+            ixx="0.0142348526057094"
+            ixy="-3.73763310100809E-08"
+            ixz="1.70703603169075E-07"
+            iyy="0.0141319978448755"
+            iyz="0.00228090337255746"
+            izz="0.00424792208583136" />
+         </inertial>
          <visual>
             <origin xyz="0 0 0" rpy="0 0 ${M_PI}" />
@@ -135,7 +135,7 @@
       </link>
       <!-- joint between lwr_2_link and lwr_3_link -->
-      <joint name="joint_2" type="revolute">
-         <parent link="link_2" />
-         <child link="link_3" />
+      <joint name="${robot_name}_joint_2" type="revolute">
+         <parent link="F_R${robot_name}_2" />
+         <child link="F_R${robot_name}_3" />
          <limit lower="${-170 * M_PI / 180}" upper="${170 * M_PI / 180}" effort="${effort_scale * 100}" velocity="${velocity_scale * 112.5 * M_PI / 180}" />
          <dynamics friction="${f2}" damping="${d2}"/>
@@ -143,19 +143,19 @@
          <axis xyz="0 0 1" />
       </joint>
-      <link name="link_3">
-    <inertial>
-      <origin
-        xyz="-1.40921289121243E-06 -0.0233297626126898 0.11815047247629"
-        rpy="0 0 0" />
-        <mass
-          value="2.30342143971329" />
-      <inertia
-        ixx="0.0156098024078732"
-        ixy="4.75479645197283E-08"
-        ixz="1.17852233217589E-07"
-        iyy="0.0153476851366831"
-        iyz="-0.00319215869825882"
-        izz="0.0044071430916942" />
-    </inertial>
+      <link name="F_R${robot_name}_3">
+         <inertial>
+            <origin
+            xyz="-1.40921289121243E-06 -0.0233297626126898 0.11815047247629"
+            rpy="0 0 0" />
+            <mass
+               value="2.30342143971329" />
+            <inertia
+            ixx="0.0156098024078732"
+            ixy="4.75479645197283E-08"
+            ixz="1.17852233217589E-07"
+            iyy="0.0153476851366831"
+            iyz="-0.00319215869825882"
+            izz="0.0044071430916942" />
+         </inertial>
          <visual>
             <origin xyz="0 0 0" rpy="0 0 ${M_PI}" />
@@ -173,7 +173,7 @@
       </link>
       <!-- joint between lwr_3_link and lwr_4_link -->
-      <joint name="joint_3" type="revolute">
-         <parent link="link_3" />
-         <child link="link_4" />
+      <joint name="${robot_name}_joint_3" type="revolute">
+         <parent link="F_R${robot_name}_3" />
+         <child link="F_R${robot_name}_4" />
          <limit lower="${-120 * M_PI / 180}" upper="${120 * M_PI / 180}" effort="${effort_scale * 100}" velocity="${velocity_scale * 112.5 * M_PI / 180}" />
          <dynamics friction="${f3}" damping="${d3}"/>
@@ -181,19 +181,19 @@
          <axis xyz="0 1 0" />
       </joint>
-      <link name="link_4">
-    <inertial>
-      <origin
-        xyz="1.12239473548659E-07 0.0327442387470235 0.073658815701594"
-        rpy="0 0 0" />
-        <mass
-          value="2.30343586527606" />
-      <inertia
-        ixx="0.0142336552604204"
-        ixy="-5.89296043886227E-08"
-        ixz="-1.568273589226E-07"
-        iyy="0.0141315528954361"
-        iyz="-0.00228056254422505"
-        izz="0.00424816761410708" />
-    </inertial>
+      <link name="F_R${robot_name}_4">
+         <inertial>
+            <origin
+            xyz="1.12239473548659E-07 0.0327442387470235 0.073658815701594"
+            rpy="0 0 0" />
+            <mass
+               value="2.30343586527606" />
+            <inertia
+            ixx="0.0142336552604204"
+            ixy="-5.89296043886227E-08"
+            ixz="-1.568273589226E-07"
+            iyy="0.0141315528954361"
+            iyz="-0.00228056254422505"
+            izz="0.00424816761410708" />
+         </inertial>
          <visual>
             <origin xyz="0 0 0" rpy="0 0 ${M_PI}" />
@@ -211,7 +211,7 @@
       </link>
       <!-- joint between lwr_4_link and lwr_5_link -->
-      <joint name="joint_4" type="revolute">
-         <parent link="link_4" />
-         <child link="link_5" />
+      <joint name="${robot_name}_joint_4" type="revolute">
+         <parent link="F_R${robot_name}_4" />
+         <child link="F_R${robot_name}_5" />
          <limit lower="${-170 * M_PI / 180}" upper="${170 * M_PI / 180}" effort="${effort_scale * 100}" velocity="${velocity_scale * 180.0 * M_PI / 180}" />
          <dynamics friction="${f4}" damping="${d4}"/>
@@ -219,19 +219,19 @@
          <axis xyz="0 0 1" />
       </joint>
-      <link name="link_5">
-    <inertial>
-      <origin
-        xyz="-6.00824789920296E-07 0.0207751869661564 0.0862053948486382"
-        rpy="0 0 0" />
-        <mass
-          value="1.60059828363332" />
-      <inertia
-        ixx="0.00880806620496216"
-        ixy="1.22820321842462E-07"
-        ixz="-5.66844221164893E-08"
-        iyy="0.00813520145401624"
-        iyz="0.00261443543508601"
-        izz="0.00359712267754715" />
-    </inertial>
+      <link name="F_R${robot_name}_5">
+         <inertial>
+            <origin
+            xyz="-6.00824789920296E-07 0.0207751869661564 0.0862053948486382"
+            rpy="0 0 0" />
+            <mass
+               value="1.60059828363332" />
+            <inertia
+            ixx="0.00880806620496216"
+            ixy="1.22820321842462E-07"
+            ixz="-5.66844221164893E-08"
+            iyy="0.00813520145401624"
+            iyz="0.00261443543508601"
+            izz="0.00359712267754715" />
+         </inertial>
          <visual>
             <origin xyz="0 0 0" rpy="0 0 ${M_PI}" />
@@ -249,7 +249,7 @@
       </link>
       <!-- joint between lwr_5_link and lwr_6_link -->
-      <joint name="joint_5" type="revolute">
-         <parent link="link_5" />
-         <child link="link_6" />
+      <joint name="${robot_name}_joint_5" type="revolute">
+         <parent link="F_R${robot_name}_5" />
+         <child link="F_R${robot_name}_6" />
          <limit lower="${-120 * M_PI / 180}" upper="${120 * M_PI / 180}" effort="${effort_scale * 30}" velocity="${velocity_scale * 112.5 * M_PI / 180}" />
          <dynamics friction="${f5}" damping="${d5}"/>
@@ -257,19 +257,19 @@
          <axis xyz="0 -1 0" />
       </joint>
-      <link name="link_6">
-    <inertial>
-      <origin
-        xyz="-2.64519244286276E-08 -0.00451753627467652 -0.00295324741635017"
-        rpy="0 0 0" />
-        <mass
-          value="1.49302436988808" />
-        <inertia
-          ixx="0.0298541138330797"
-          ixy="-3.97658663154265E-09"
-          ixz="-1.71667243685877E-09"
-          iyy="0.0299834927882566"
-          iyz="-2.53647350791604E-05"
-          izz="0.0323627047307316" />
-    </inertial>
+      <link name="F_R${robot_name}_6">
+         <inertial>
+            <origin
+            xyz="-2.64519244286276E-08 -0.00451753627467652 -0.00295324741635017"
+            rpy="0 0 0" />
+            <mass
+               value="1.49302436988808" />
+            <inertia
+               ixx="0.0298541138330797"
+               ixy="-3.97658663154265E-09"
+               ixz="-1.71667243685877E-09"
+               iyy="0.0299834927882566"
+               iyz="-2.53647350791604E-05"
+               izz="0.0323627047307316" />
+         </inertial>
          <visual>
             <origin xyz="0 0 0" rpy="0 0 ${M_PI}" />
@@ -287,7 +287,7 @@
       </link>
       <!-- joint between lwr_6_link and lwr_7_link -->
-      <joint name="joint_6" type="revolute">
-         <parent link="link_6" />
-         <child link="link_7" />
+      <joint name="${robot_name}_joint_6" type="revolute">
+         <parent link="F_R${robot_name}_6" />
+         <child link="F_R${robot_name}_7" />
          <limit lower="${-170 * M_PI / 180}" upper="${170 * M_PI / 180}" effort="${effort_scale * 30}" velocity="${velocity_scale * 112.5 * M_PI / 180}" />
          <dynamics friction="${f6}" damping="${d6}"/>
@@ -295,19 +295,19 @@
          <axis xyz="0 0 1" />
       </joint>
-      <link name="link_7">
-    <inertial>
-      <origin
-        xyz="2.77555756156289E-17 1.11022302462516E-16 -0.015814675599801"
-        rpy="0 0 0" />
-        <mass
-          value="0.108688241139613" />
-        <inertia
-          ixx="4.17908737998876E-02"
-          ixy="0"
-          ixz="0"
-          iyy="4.17908737998876E-02"
-          iyz="0"
-          izz="7.00756879151782E-02" />
-    </inertial>
+      <link name="F_R${robot_name}_7">
+         <inertial>
+            <origin
+            xyz="2.77555756156289E-17 1.11022302462516E-16 -0.015814675599801"
+            rpy="0 0 0" />
+            <mass
+               value="0.108688241139613" />
+            <inertia
+               ixx="4.17908737998876E-02"
+               ixy="0"
+               ixz="0"
+               iyy="4.17908737998876E-02"
+               iyz="0"
+               izz="7.00756879151782E-02" />
+         </inertial>
          <visual>
             <origin xyz="0 0 0" rpy="0 0 ${M_PI}" />

Commit message: Add end-effector link

File: urdf/lwr.urdf.xacro (robot description, xacro)
@@ -324,4 +324,11 @@
          </collision>
       </link>
+      <joint name="${robot_name}_joint_ee" type="fixed">
+         <parent link="F_R${robot_name}_7"/>
+         <child link="F_RE${robot_name}"/>
+         <origin xyz="0 0 0" rpy="0 0 0"/>
+      </joint>
+      <link name="F_RE${robot_name}">
+      </link>
    </xacro:macro>
 </robot>
